File: tc2030-swd-adapter.kicad_sch (KiCad schematic)
At the start: 2 parts, among them J1 TC2030, J2 JLINK-Interface

Commit message: Finish pcb
Parts:
- added C1, C2: 1u, Capacitor_SMD:C_0603_1608Metric, symbol Device:C_Small
- added D1: 1N41008, Diode_SMD:D_SOD-123, symbol Device:D_Small
- added D2: LED_Small, LED_SMD:LED_0603_1608Metric, symbol Device:LED_Small
- added J3: Conn_01x03, Connector_PinHeader_2.54mm:PinHeader_1x03_P2.54mm_Vertical, symbol Connector_Generic:Conn_01x03
- added J4: Conn_01x02, Connector_PinHeader_2.54mm:PinHeader_1x02_P2.54mm_Vertical, symbol Connector_Generic:Conn_01x02
- added J5: TC2030, Connector_IDC:IDC-Header_2x03_P2.54mm_Vertical, symbol tc2030-adapter:Conn_ARM_SWD_TagConnect_TC2030
- added JP1, JP2: Jumper_3_Open, Connector_PinHeader_2.54mm:PinHeader_1x03_P2.54mm_Vertical, symbol Jumper:Jumper_3_Open
- added R1: 100, Resistor_SMD:R_0603_1608Metric, symbol Device:R_Small
- added R2: 1k, Resistor_SMD:R_0603_1608Metric, symbol Device:R_Small
- added SW1: B3U-1000P, Button_Switch_SMD:SW_SPST_B3U-1000P, symbol Switch:SW_Push
- added U1: RT9080-33GJ5, Package_TO_SOT_SMD:TSOT-23-5, symbol tc2030-adapter:RT9080-33GJ5
- J1: footprint Connector:Tag-Connect_TC2030-IDC-NL_2x03_P1.27mm_Vertical -> Connector_IDC:IDC-Header_2x03_P2.54mm_Vertical
- J2: footprint (none) -> Connector_PinSocket_2.54mm:PinSocket_2x10_P2.54mm_Horizontal
Connections:
- net GND: now also J1.5 (GND), C1.2, C2.2, D2.1 (K), J3.1 (Pin_1), J4.1 (Pin_1), J5.5 (GND), R1.2, U1.2 (GND)
- net SWCLK: now also J1.4 (SWCLK), J5.4 (SWCLK)
- net SWDIO: now also J1.2 (SWDIO), J5.2 (SWDIO)
- net SWO: now also J1.6 (SWO)
- net VTref: now also D1.1 (K)
- net nRST: now also J1.3 (~{RESET}), SW1.1
- net VCC: now reaches J1.1 (VCC)
- net VCC: now also J5.1 (VCC), JP2.2 (C)
- net 5V renamed +5V
- net +5V: now also C1.1, JP1.1 (A), JP2.1 (A), R2.1, U1.1 (Vin), U1.3 (EN)
- new net: D2.2 (A), R2.2
- new net: R1.1, SW1.2
- new net +3V3: C2.1, JP1.3 (B), JP2.3 (B), U1.5 (Vout)
- new net RX: J3.3 (Pin_3), J5.3 (RX)
- new net TX: J3.2 (Pin_2), J5.6 (TX)
- new net VTref_in: D1.2 (A), J4.2 (Pin_2), JP1.2 (C)
Other:
- title: (none) -> TC2030-JLINK-Adapter
- moved on the sheet: J1, J2

Commit message: Add UART to JLINK
Connections:
- net RX is gone; now on net JLINK_TX: J3.3 (Pin_3), J5.3 (RX)
- net TX is gone; now on net JLINK_RX: J3.2 (Pin_2), J5.6 (TX)
- net JLINK_RX: now reaches J2.17 (Pin_17)
- net JLINK_TX: now reaches J2.5 (Pin_5)
- no-connect marks 5 -> 3
Changed lines of the file:
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@@
   (junction (at 87.63 104.14) (diameter 0) (color 0 0 0 0)
   )
-  (no_connect (at 104.14 93.98))
   (no_connect (at 104.14 101.6))
   (no_connect (at 91.44 88.9))
   (no_connect (at 104.14 91.44))
-  (no_connect (at 104.14 109.22))
   (wire (pts (xy 87.63 101.6) (xy 87.63 99.06))
     (stroke (width 0) (type default))
@@
     (stroke (width 0) (type default))
   )
+  (wire (pts (xy 222.25 110.49) (xy 238.76 110.49))
+    (stroke (width 0) (type default))
+  )
   (wire (pts (xy 87.63 99.06) (xy 87.63 96.52))
     (stroke (width 0) (type default))
@@
     (stroke (width 0) (type default))
   )
+  (wire (pts (xy 104.14 93.98) (xy 113.03 93.98))
+    (stroke (width 0) (type default))
+  )
   (wire (pts (xy 87.63 106.68) (xy 87.63 104.14))
     (stroke (width 0) (type default))
@@
     (stroke (width 0) (type default))
   )
+  (wire (pts (xy 104.14 109.22) (xy 113.03 109.22))
+    (stroke (width 0) (type default))
+  )
   (wire (pts (xy 87.63 109.22) (xy 87.63 111.76))
     (stroke (width 0) (type default))
@@
     (stroke (width 0) (type default))
   )
+  (wire (pts (xy 222.25 100.33) (xy 238.76 100.33))
+    (stroke (width 0) (type default))
+  )
   (wire (pts (xy 87.63 93.98) (xy 87.63 91.44))
     (stroke (width 0) (type default))
@@
     (stroke (width 0) (type default))
   )
-  (wire (pts (xy 222.25 100.33) (xy 229.87 100.33))
-    (stroke (width 0) (type default))
-  )
   (wire (pts (xy 191.77 100.33) (xy 199.39 100.33))
     (stroke (width 0) (type default))
@@
     (stroke (width 0) (type default))
   )
-  (wire (pts (xy 222.25 110.49) (xy 229.87 110.49))
-    (stroke (width 0) (type default))
-  )
   (wire (pts (xy 86.36 59.69) (xy 88.9 59.69))
     (stroke (width 0) (type default))
@@
     (effects (font (size 1.27 1.27)) (justify left bottom))
   )
+  (label "JLINK_TX" (at 238.76 100.33 180) (fields_autoplaced)
+    (effects (font (size 1.27 1.27)) (justify right bottom))
+  )
+  (label "JLINK_TX" (at 113.03 93.98 180) (fields_autoplaced)
+    (effects (font (size 1.27 1.27)) (justify right bottom))
+  )
   (label "TX" (at 203.2 69.85 0) (fields_autoplaced)
     (effects (font (size 1.27 1.27)) (justify left bottom))
@@
     (effects (font (size 1.27 1.27)) (justify right bottom))
   )
+  (label "JLINK_RX" (at 238.76 110.49 180) (fields_autoplaced)
+    (effects (font (size 1.27 1.27)) (justify right bottom))
+  )
   (label "VTref_in" (at 168.91 67.31 0) (fields_autoplaced)
     (effects (font (size 1.27 1.27)) (justify left bottom))
@@
     (effects (font (size 1.27 1.27)) (justify right bottom))
   )
+  (label "JLINK_RX" (at 113.03 109.22 180) (fields_autoplaced)
+    (effects (font (size 1.27 1.27)) (justify right bottom))
+  )
